Commit message: stereo depth setting has been included

File: urdf/system_hss.urdf.xacro (robot description, xacro)
@@ -6,4 +6,26 @@
 <xacro:arg name="use_gazebo" default="false" />
 <link name="camera_spin_link">
+<inertial>
+  <origin xyz="0 0 0" rpy="0 0 0"/>
+  <mass value="3.43533e-05"/>
+  <inertia
+    ixx="1.03260e-10" ixy="0" ixz="0"
+    iyy="1.03260e-10" iyz="0"
+    izz="6.33819e-11"/>
+</inertial>
+  <visual>
+  <origin xyz="0 0 0" rpy="0 0 0"/>
+    <geometry>
+      <cylinder length="0.002" radius="0.0015"/>
+    </geometry>
+  </visual>
+  <collision>
+  <origin xyz="0 0 0" rpy="0 0 0"/>
+    <geometry>
+      <cylinder length="0.005" radius="0.0015"/>
+    </geometry>
+  </collision>
+</link>
+<link name="left_camera_spin_link">
 <inertial>
   <origin xyz="0 0 0" rpy="0 0 0"/>
@@ -358,7 +380,12 @@
     <origin xyz="0.005 0 0.008" rpy="0 3.1415 0"/> <!-- 90° pitch yukarı baktırıyor -->
   </joint>
+<joint name="left_camera_joint" type="fixed">
+    <parent link="camera_link"/>
+    <child link="left_camera_spin_link"/>
+    <origin xyz="-0.055 0 0.008" rpy="0 3.1415 0"/> <!-- 90° pitch yukarı baktırıyor -->
+  </joint>
 <!-- ///////////////////////// gazebo  parameters////////////////////////////-->
     <gazebo reference="camera_spin_link">
-        <sensor name="camera" type="camera">
+        <sensor name="right_camera" type="camera">
          <pose>0 0 0 0 1.57 1.57</pose> <!-- roll pitch yaw -->
             <always_on>true</always_on>
@@ -377,8 +404,34 @@
             </clip>
             </camera>
-            <plugin filename="gz-sim-sensors-system"
-            name="gz::sim::systems::Sensors"/>
-            <topic>camera/image</topic> <!-- Gazebo topic -->
+            <!-- <plugin filename="gz-sim-sensors-system"
+            name="gz::sim::systems::Sensors"/> -->
+            <topic>camera0/image</topic> <!-- Gazebo topic -->
         </sensor>
     </gazebo>
+    <gazebo reference="left_camera_spin_link">
+        <sensor name="left_camera" type="camera">
+         <pose>0 0 0 0 1.57 1.57</pose> <!-- roll pitch yaw -->
+            <always_on>true</always_on>
+            <update_rate>60</update_rate>        <!-- FPS -->
+            <visualize>true</visualize>
+            <camera>
+            <horizontal_fov>1.047</horizontal_fov> <!-- 60 derece -->
+            <image>
+                <width>640</width>
+                <height>480</height>
+                <format>R8G8B8</format>
+            </image>
+            <clip>
+                <near>0.1</near>
+                <far>100</far>
+            </clip>
+            </camera>
+            <!-- <plugin filename="gz-sim-sensors-system"
+            name="gz::sim::systems::Sensors"/> -->
+            <topic>camera1/image</topic>
+        </sensor>
+    </gazebo>
+    <plugin name='gz::sim::systems::Sensors' filename='gz-sim-sensors-system'>
+    <render_engine>ogre</render_engine>
+</plugin>
 </robot>
